File: lm386_amp.kicad_pcb (KiCad board)
At the start: 2 copper layers, 45.7 x 33 mm, 18 parts, among them J1 Conn_01x02_Pin, J2 Conn_01x02_Pin, J3 Conn_01x02_Pin, U1 LM386

Commit message: update
Parts:
- moved C2 4.17 mm to (85.4, 69.6), turned to 180 degrees
- moved C6 3.81 mm to (86.4, 87.6), turned to -90 degrees
- moved G*** 2.84 mm to (99.1, 90.2)
- moved R2 1.27 mm to (81.3, 87.6)
- moved C1 1.27 mm to (77.5, 78.7)
Routing:
- net Net-(U1-+): track 13.4 -> 9.52 mm
- net Net-(C1-Pad1): track 10.2 -> 7.44 mm
- net Net-(U1-BYPASS): track 9.32 -> 6.60 mm
- net +9V: track 40.9 -> 39.2 mm
- net Net-(C1-Pad2): track 6.63 -> 5.36 mm
- net Net-(J3-Pin_1): track 8.67 -> 7.44 mm
Changed lines of the file:
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@@
   )
   (footprint "LOGO" (layer "F.Cu")
-    (at 101.6 88.9)
+    (at 99.06 90.17)
     (attr board_only exclude_from_pos_files exclude_from_bom)
     (fp_text reference "G***" (at 0 0) (layer "F.SilkS") hide
@@
   )
   (footprint "Capacitor_THT:C_Radial_D6.3mm_H5.0mm_P2.50mm" (layer "F.Cu")
-    (at 86.4 91.44)
+    (at 86.36 87.63 -90)
     (descr "C, Radial series, Radial, pin pitch=2.50mm, diameter=6.3mm, height=5mm, Non-Polar Electrolytic Capacitor")
     (tags "C Radial series Radial pin pitch 2.50mm diameter 6.3mm height 5mm Non-Polar Electrolytic Capacitor")
@@
     (property "ki_keywords" "capacitor cap")
     (attr through_hole)
-    (fp_text reference "C6" (at 1.25 -4.4) (layer "F.SilkS")
+    (fp_text reference "C6" (at 1.25 -4.4 90) (layer "F.SilkS")
         (effects (font (size 1 1) (thickness 0.15)))
     )
-    (fp_text value "4.7μF" (at 1.25 4.4) (layer "F.Fab")
+    (fp_text value "4.7μF" (at 1.25 4.4 90) (layer "F.Fab")
         (effects (font (size 1 1) (thickness 0.15)))
     )
-    (fp_text user "${REFERENCE}" (at 1.25 0) (layer "F.Fab")
+    (fp_text user "${REFERENCE}" (at 1.25 0 90) (layer "F.Fab")
         (effects (font (size 1 1) (thickness 0.15)))
     )
@@
     (fp_circle (center 1.25 0) (end 4.4 0)
       (stroke (width 0.1) (type solid)) (fill none) (layer "F.Fab"))
-    (pad "1" thru_hole circle (at 0 0) (size 1.6 1.6) (drill 0.8) (layers "*.Cu" "*.Mask")
+    (pad "1" thru_hole circle (at 0 0 270) (size 1.6 1.6) (drill 0.8) (layers "*.Cu" "*.Mask")
       (net 6 "Net-(U1-+)") (pintype "passive"))
-    (pad "2" thru_hole circle (at 2.5 0) (size 1.6 1.6) (drill 0.8) (layers "*.Cu" "*.Mask")
+    (pad "2" thru_hole circle (at 2.5 0 270) (size 1.6 1.6) (drill 0.8) (layers "*.Cu" "*.Mask")
       (net 7 "Net-(J3-Pin_1)") (pintype "passive"))
     (model "${KICAD6_3DMODEL_DIR}/Capacitor_THT.3dshapes/C_Radial_D6.3mm_H5.0mm_P2.50mm.wrl"
@@
   )
   (footprint "Capacitor_THT:CP_Radial_D7.5mm_P2.50mm" (layer "F.Cu")
-    (at 81.32 68.58)
+    (at 85.361395 69.6 180)
     (descr "CP, Radial series, Radial, pin pitch=2.50mm, , diameter=7.5mm, Electrolytic Capacitor")
     (tags "CP Radial series Radial pin pitch 2.50mm  diameter 7.5mm Electrolytic Capacitor")
@@
     (property "ki_keywords" "cap capacitor")
     (attr through_hole)
-    (fp_text reference "C2" (at -5.12 -2.54) (layer "F.SilkS")
+    (fp_text reference "C2" (at 5.351395 3.56) (layer "F.SilkS")
         (effects (font (size 1 1) (thickness 0.15)))
     )
-    (fp_text value "C_Polarized_Small" (at 1.25 5) (layer "F.Fab")
+    (fp_text value "C_Polarized_Small" (at 1.25 3.73) (layer "F.Fab")
         (effects (font (size 1 1) (thickness 0.15)))
     )
@@
     (fp_circle (center 1.25 0) (end 5 0)
       (stroke (width 0.1) (type solid)) (fill none) (layer "F.Fab"))
-    (pad "1" thru_hole rect (at 0 0) (size 1.6 1.6) (drill 0.8) (layers "*.Cu" "*.Mask")
+    (pad "1" thru_hole rect (at 0 0 180) (size 1.6 1.6) (drill 0.8) (layers "*.Cu" "*.Mask")
       (net 3 "Net-(U1-BYPASS)") (pintype "passive"))
-    (pad "2" thru_hole circle (at 2.5 0) (size 1.6 1.6) (drill 0.8) (layers "*.Cu" "*.Mask")
+    (pad "2" thru_hole circle (at 2.5 0 180) (size 1.6 1.6) (drill 0.8) (layers "*.Cu" "*.Mask")
       (net 4 "GND") (pintype "passive"))
     (model "${KICAD6_3DMODEL_DIR}/Capacitor_THT.3dshapes/CP_Radial_D7.5mm_P2.50mm.wrl"
@@
   )
   (footprint "Capacitor_THT:CP_Radial_D5.0mm_P2.50mm" (layer "F.Cu")
-    (at 76.2 78.74 90)
+    (at 77.47 78.74 90)
     (descr "CP, Radial series, Radial, pin pitch=2.50mm, , diameter=5mm, Electrolytic Capacitor")
     (tags "CP Radial series Radial pin pitch 2.50mm  diameter 5mm Electrolytic Capacitor")
@@
   )
   (footprint "Resistor_THT:R_Axial_DIN0207_L6.3mm_D2.5mm_P10.16mm_Horizontal" (layer "F.Cu")
-    (at 81.28 88.9 180)
+    (at 81.28 87.63 180)
     (descr "Resistor, Axial_DIN0207 series, Axial, Horizontal, pin pitch=10.16mm, 0.25W = 1/4W, length*diameter=6.3*2.5mm^2, http://cdn-reichelt.de/documents/datenblatt/B400/1_4W%23YAG.pdf")
     (tags "Resistor Axial_DIN0207 series Axial Horizontal pin pitch 10.16mm 0.25W = 1/4W length 6.3mm diameter 2.5mm")
@@
   (gr_rect (start 68.58 63.5) (end 114.3 96.52)
     (stroke (width 0.1) (type default)) (fill none) (layer "Edge.Cuts"))
-  (segment (start 76.2 81.28) (end 78.74 83.82) (width 0.8) (layer "B.Cu") (net 1))
-  (segment (start 78.74 83.82) (end 82.81 83.82) (width 0.8) (layer "B.Cu") (net 1))
-  (segment (start 76.2 78.74) (end 76.2 81.28) (width 0.8) (layer "B.Cu") (net 1))
+  (segment (start 82.55 83.82) (end 77.47 78.74) (width 0.8) (layer "B.Cu") (net 1))
+  (segment (start 82.81 83.82) (end 82.55 83.82) (width 0.8) (layer "B.Cu") (net 1))
   (segment (start 82.77 76.24) (end 82.81 76.2) (width 0.8) (layer "B.Cu") (net 2))
-  (segment (start 76.2 76.24) (end 82.77 76.24) (width 0.8) (layer "B.Cu") (net 2))
-  (segment (start 81.28 72.13) (end 81.28 71.12) (width 0.8) (layer "B.Cu") (net 3))
-  (segment (start 81.32 71.08) (end 81.32 68.58) (width 0.8) (layer "B.Cu") (net 3))
-  (segment (start 81.28 71.12) (end 81.32 71.08) (width 0.8) (layer "B.Cu") (net 3))
-  (segment (start 85.35 76.2) (end 81.28 72.13) (width 0.8) (layer "B.Cu") (net 3))
+  (segment (start 77.47 76.24) (end 82.77 76.24) (width 0.8) (layer "B.Cu") (net 2))
+  (segment (start 85.361395 76.188605) (end 85.35 76.2) (width 0.8) (layer "B.Cu") (net 3))
+  (segment (start 85.361395 69.6) (end 85.361395 76.188605) (width 0.8) (layer "B.Cu") (net 3))
   (segment (start 93.9 83.82) (end 93.98 83.74) (width 0.8) (layer "B.Cu") (net 4))
   (segment (start 99.06 71.12) (end 99.06 66.12) (width 0.8) (layer "B.Cu") (net 5))
   (segment (start 99.06 66.12) (end 99.14 66.04) (width 0.8) (layer "B.Cu") (net 5))
-  (segment (start 86.36 88.9) (end 86.4 88.94) (width 0.8) (layer "B.Cu") (net 6))
-  (segment (start 86.36 88.9) (end 83.86 88.9) (width 0.8) (layer "B.Cu") (net 6))
-  (segment (start 87.89 83.82) (end 87.89 87.37) (width 0.8) (layer "B.Cu") (net 6))
-  (segment (start 87.89 87.37) (end 86.36 88.9) (width 0.8) (layer "B.Cu") (net 6))
-  (segment (start 83.86 88.9) (end 82.81 88.9) (width 0.8) (layer "B.Cu") (net 6))
-  (segment (start 82.81 88.9) (end 81.28 88.9) (width 0.8) (layer "B.Cu") (net 6))
-  (segment (start 86.4 88.94) (end 86.4 91.44) (width 0.8) (layer "B.Cu") (net 6))
-  (segment (start 86.36 93.98) (end 81.28 93.98) (width 0.8) (layer "B.Cu") (net 7))
-  (segment (start 88.9 91.44) (end 86.36 93.98) (width 0.8) (layer "B.Cu") (net 7))
+  (segment (start 87.89 83.82) (end 87.89 86.1) (width 0.8) (layer "B.Cu") (net 6))
+  (segment (start 87.89 86.1) (end 86.36 87.63) (width 0.8) (layer "B.Cu") (net 6))
+  (segment (start 81.28 87.63) (end 86.36 87.63) (width 0.8) (layer "B.Cu") (net 6))
+  (segment (start 83.82 93.98) (end 81.28 93.98) (width 0.8) (layer "B.Cu") (net 7))
+  (segment (start 86.36 90.13) (end 86.36 91.44) (width 0.8) (layer "B.Cu") (net 7))
+  (segment (start 86.36 91.44) (end 83.82 93.98) (width 0.8) (layer "B.Cu") (net 7))
   (segment (start 111.72 73.7) (end 111.76 73.66) (width 0.8) (layer "B.Cu") (net 8))
   (segment (start 106.68 73.7) (end 111.72 73.7) (width 0.8) (layer "B.Cu") (net 8))
+  (segment (start 76.58 68.2) (end 90.15 68.2) (width 0.8) (layer "B.Cu") (net 9))
   (segment (start 87.89 76.2) (end 90.43 78.74) (width 0.8) (layer "B.Cu") (net 9))
   (segment (start 87.89 72.13) (end 87.89 76.2) (width 0.8) (layer "B.Cu") (net 9))
+  (segment (start 71.12 73.66) (end 76.58 68.2) (width 0.8) (layer "B.Cu") (net 9))
   (segment (start 91.56 69.61) (end 90.41 69.61) (width 0.8) (layer "B.Cu") (net 9))
-  (segment (start 78.6 66.18) (end 71.12 73.66) (width 0.8) (layer "B.Cu") (net 9))
-  (segment (start 88.13 66.18) (end 78.6 66.18) (width 0.8) (layer "B.Cu") (net 9))
   (segment (start 90.41 69.61) (end 87.89 72.13) (width 0.8) (layer "B.Cu") (net 9))
-  (segment (start 91.56 69.61) (end 88.13 66.18) (width 0.8) (layer "B.Cu") (net 9))
+  (segment (start 90.15 68.2) (end 91.56 69.61) (width 0.8) (layer "B.Cu") (net 9))
   (segment (start 90.43 78.74) (end 93.98 78.74) (width 0.8) (layer "B.Cu") (net 9))
   (segment (start 99.06 76.2) (end 101.6 73.66) (width 0.8) (layer "B.Cu") (net 10))
@@
     (connect_pads (clearance 0.5))
     (min_thickness 0.25) (filled_areas_thickness no)
-    (fill (thermal_gap 0.5) (thermal_bridge_width 0.5))
+    (fill yes (thermal_gap 0.5) (thermal_bridge_width 0.5))
     (polygon
       (pts
